Commit message: Set table, cup for cafe manipulator using URDF

File: examples/rsc/kinova/urdf/kinova.urdf (robot description, URDF)
Before this commit: robot kinova, 10 links, 9 joints
Links:
- added link table_leg; visual cylinder length=0.5 radius=0.07
- added link table_plate; visual cylinder length=0.05 radius=0.3
Joints:
- added joint table_joint: type fixed, parent table_leg, child table_plate, origin xyz=0 0 0.5 rpy=0 0 0
- added joint world_joint: type fixed, parent world, child table_leg, origin xyz=0 0 0 rpy=0 0 0
- joint kinova_joint_base: origin xyz=0 0 0 rpy=0 0 0 -> xyz=0 0 0.05 rpy=0 0 0; parent world -> table_plate

Commit message: Added Kinova arm & table collision

File: examples/rsc/kinova/urdf/kinova.urdf (robot description, URDF)
Before this commit: robot kinova, 12 links, 11 joints
Links:
- link kinova_link_2: geometry collision box size=0.06 0.45 0.015; visual mesh filename=../meshes/arm.dae
- link kinova_link_3: geometry collision box size=0.06 0.22 0.015; visual mesh filename=../meshes/forearm.dae
- link kinova_link_5: geometry collision box size=0.05 0.15 0.02; visual mesh filename=../meshes/ring_small.STL
- link kinova_link_6: geometry collision box size=0.075 0.075 0.075; visual mesh filename=../meshes/hand_3finger.dae
- link kinova_link_base: geometry collision cylinder length=0.15 radius=0.035; visual mesh filename=../meshes/base.dae
- link table_leg: geometry collision cylinder length=0.5 radius=0.07; visual cylinder length=0.5 radius=0.07
- link table_plate: geometry collision cylinder length=0.05 radius=0.3; visual cylinder length=0.05 radius=0.3

Commit message: Edited URDF Collision(2)

File: examples/rsc/kinova/urdf/kinova.urdf (robot description, URDF)
Before this commit: robot kinova, 12 links, 11 joints
Links:
- link kinova_link_1: geometry collision cylinder length=0.14 radius=0.015; visual mesh filename=../meshes/ring_big.STL
- link kinova_link_4: geometry collision cylinder length=0.03 radius=0.03; visual mesh filename=../meshes/ring_small.STL

Commit message: Cup holder project?

File: examples/rsc/kinova/urdf/kinova.urdf (robot description, URDF)
Before this commit: robot kinova, 12 links, 11 joints
Links:
- link kinova_link_6: geometry collision box size=0.1 0.1 0.1; visual mesh filename=../meshes/hand_3finger.dae

Commit message: Hit the ball. Collision problem solved.

File: examples/rsc/kinova/urdf/kinova.urdf (robot description, URDF)
Before this commit: robot kinova, 12 links, 11 joints
Links:
- link kinova_link_6: geometry collision box size=0.07 0.07 0.07; visual mesh filename=../meshes/hand_3finger.dae
