Commit message: Set Floating base Cup offset to Zero.

File: examples/rsc/kinova/urdf/cup.urdf (robot description, URDF)
Before this commit: robot cup, 2 links, 1 joints
Links:
- link cup: mass 1.293 -> 0.05

Commit message: changed obstacle into cup.(for job PT)

File: examples/rsc/kinova/urdf/cup.urdf (robot description, URDF)
Before this commit: robot cup, 2 links, 1 joints
Links:
- link cup: geometry collision sphere radius=0.06; visual sphere radius=0.06
